File: pcb/v1/hava_routed.kicad_pcb (KiCad board)
At the start: 2 copper layers, 50 x 56 mm, 23 parts, among them J1 USB_C_Receptacle_USB2.0_16P, J2 Conn_01x08, SW1 SW_Push, SW2 SW_Push, SW3 SW_Push, U1 ESP32-C3-WROOM-02, U2 AP2112K-3.3, U3 BME280, U4 USBLC6-2SC6

Commit message: Kutu (FreeCAD), ESP32'siz PC demosu, ikinci datasheet denetimi ve süreç notları
- case/: kartın ölçülerini KiCad'den okuyup FreeCAD ile kutu ve kapak üretir,
  parçalı 3D kart modeliyle çakışma kontrolü yapar (çakışma 0).
- firmware/pc_demo: gerçek Open-Meteo verisi + firmware'in gerçek ekran ve
  sensör hesap kodu ile ESP32 olmadan ekran görüntüsü üretir.
- Kart: IO2 ve IO8 pull-up, BME280 için ikinci 100 nF (datasheet denetimi).
- docs/SUREC-NOTLARI.md, docs/v1/03-denetim-2.md, çalışma günlüğü güncellendi.
Parts:
- added C7: 100nF, C_0402_1005Metric, F.Cu at (139.0, 141.2)
- added R8: 10k, R_0402_1005Metric, F.Cu at (137.0, 122.2)
- added R9: 10k, R_0402_1005Metric, F.Cu at (113.0, 116.2)
Connections:
- U1 pad 16: (no net) -> N$3
- U1 pad 7: (no net) -> N$4
Routing:
- net LCD_SCK: track 76.8 -> 31.9 mm
- net N$3: track 0.00 -> 34.5 mm
- net +3V3: track 134.0 -> 164.2 mm, vias 1 -> 4
- net EN: track 40.4 -> 55.5 mm
- net GND: track 207.0 -> 197.6 mm
- net N$4: track 0.00 -> 7.77 mm
- net BOOT: track 38.6 -> 31.5 mm, vias 2 -> 0
- net USB_DM: track 48.3 -> 54.1 mm, vias 0 -> 2
- net N$1: track 10.3 -> 15.2 mm
- net BTN_IO: track 58.8 -> 53.8 mm
- net N$2: track 10.9 -> 15.7 mm, vias 0 -> 2
- net +5V: track 32.4 -> 37.2 mm, vias 3 -> 4
- net USB_DP: track 55.4 -> 52.6 mm, vias 2 -> 0
- net I2C_SDA: track 67.2 -> 64.6 mm
- net I2C_SCL: track 59.5 -> 61.4 mm, vias 3 -> 2
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