File: pcb/main/hava.kicad_pcb (KiCad board)
At the start: 2 copper layers, 32 x 41 mm, 24 parts, among them J1 USB_C_Receptacle_USB2.0_16P, J2 Conn_01x04, SW1 SW_Push, SW2 SW_Push, U1 ESP32-C3-WROOM-02, U2 AP2112K-3.3, U4 USBLC6-2SC6

Commit message: Şematik akışı: kartlar KiCad şematiğinden kuruluyor
Önceden SKiDL netlistinden doğrudan PCB üretiliyordu, arada şematik yoktu.
Artık akış: SKiDL devre tanımı -> KiCad şematiği (hava.kicad_sch) -> ERC ->
şematikten netlist -> PCB yerleşimi -> yol çizimi -> DRC (şematik paritesiyle).

- pcb/tools/sch_gen.py: netlistten KiCad şematiği üretir (İngilizce blok başlıkları)
- pcb/tools/check.sh: şematik üretimi, ERC, netlist karşılaştırması, PDF çıktısı
- pcb/tools/relink_board.py: yolları bozmadan footprint'leri şematiğe yeniden bağlar
- İsimsiz netlere ad verildi: USB_CC1/2, IO2_PU, IO8_PU, LED_A
- Sonuç: ERC 0 hata, DRC 0 ihlal, 0 bağlanmamış pad, şematik-PCB paritesi temiz
Connections:
- net BOOT renamed /BOOT
- net EN renamed /EN
- net I2C_SCL renamed /I2C_SCL
- net I2C_SDA renamed /I2C_SDA
- net LED_IO renamed /LED_IO
- net N$1 renamed /USB_CC1
- net N$2 renamed /USB_CC2
- net N$3 renamed /IO2_PU
- net N$4 renamed /IO8_PU
- net N$5 renamed /LED_A
- net USB_DM renamed /USB_DM
- net USB_DP renamed /USB_DP
- J1 pad A8: (no net) -> unconnected-(J1-SBU1-PadA8)
- J1 pad B8: (no net) -> unconnected-(J1-SBU2-PadB8)
- U1 pad 10: (no net) -> unconnected-(U1-IO10-Pad10)
- U1 pad 12: (no net) -> unconnected-(U1-IO21/TXD-Pad12)
- U1 pad 15: (no net) -> unconnected-(U1-IO3-Pad15)
- U1 pad 17: (no net) -> unconnected-(U1-IO1-Pad17)
- U1 pad 18: (no net) -> unconnected-(U1-IO0-Pad18)
- U1 pad 5: (no net) -> unconnected-(U1-IO6-Pad5)
- U1 pad 6: (no net) -> unconnected-(U1-IO7-Pad6)
- U2 pad 4: (no net) -> unconnected-(U2-NC-Pad4)
