File: pcb/sensor/hava.kicad_pcb (KiCad board)
At the start: 2 copper layers, 14 x 16 mm, 6 parts, among them J1 Conn_01x04, U1 BME280

Commit message: Şematik akışı: kartlar KiCad şematiğinden kuruluyor
Önceden SKiDL netlistinden doğrudan PCB üretiliyordu, arada şematik yoktu.
Artık akış: SKiDL devre tanımı -> KiCad şematiği (hava.kicad_sch) -> ERC ->
şematikten netlist -> PCB yerleşimi -> yol çizimi -> DRC (şematik paritesiyle).

- pcb/tools/sch_gen.py: netlistten KiCad şematiği üretir (İngilizce blok başlıkları)
- pcb/tools/check.sh: şematik üretimi, ERC, netlist karşılaştırması, PDF çıktısı
- pcb/tools/relink_board.py: yolları bozmadan footprint'leri şematiğe yeniden bağlar
- İsimsiz netlere ad verildi: USB_CC1/2, IO2_PU, IO8_PU, LED_A
- Sonuç: ERC 0 hata, DRC 0 ihlal, 0 bağlanmamış pad, şematik-PCB paritesi temiz
Connections:
- net I2C_SCL renamed /I2C_SCL
- net I2C_SDA renamed /I2C_SDA
